Commit message: feature: añadido planeación de trayecotria, ejecutar como ros2 run antropomorfico_sim ejecutar_trayectoria --ros-args -p use_sim_time:=true

File: Robot1/codigo_fuente/antropomorfico_ws/src/antropomorfico_sim/urdf/antropomorfico.urdf (robot description, URDF)
Before this commit: robot antropomorfico_sim, 9 links, 8 joints
Joints:
- joint joint_dedoder: limit lower=0.0 upper=0.015 effort=10.0 velocity=0.05 -> lower=0.0 upper=0.015 effort=500.0 velocity=0.5
- joint joint_dedoizq: limit lower=0.0 upper=0.015 effort=10.0 velocity=0.05 -> lower=0.0 upper=0.015 effort=500.0 velocity=0.5

Commit message: feature: añadido codigos de matlab y cambios en la logica de las trayectorias

File: Robot1/codigo_fuente/antropomorfico_ws/src/antropomorfico_sim/urdf/antropomorfico.urdf (robot description, URDF)
Before this commit: robot antropomorfico_sim, 9 links, 8 joints
Joints:
- joint joint1: limit lower=-3.1416 upper=3.1416 effort=10.0 velocity=3.0 -> effort=10.0 velocity=3.0; type revolute -> continuous
