Commit message: Planos mecanicos

File: Robot4/Codigo fuente/robotica/src/scara_boceto/urdf/final.urdf (robot description, URDF)
Before this commit: robot scara_boceto, 6 links, 5 joints
Links:
- removed link ban3
- removed link est2
- removed link pris
- added link caja, mass 0.40399; collision mesh filename=package://scara_boceto/meshes/caja.STL; visual mesh filename=package://scara_boceto/meshes/caja.STL
- added link efector, mass 0.00140887146453861; collision mesh filename=package://scara_boceto/meshes/efector.STL; visual mesh filename=package://scara_boceto/meshes/efector.STL
- added link prisma, mass 0.0482530059600755; collision mesh filename=package://scara_boceto/meshes/prisma.STL; visual mesh filename=package://scara_boceto/meshes/prisma.STL
- link base_link: mass 0.311284852028824 -> 0.36928
- link rot1: mass 0.94931 -> 0.96022
- link rot2: mass 0.67755 -> 0.8275
Joints:
- removed joint ban3
- removed joint est2
- removed joint pris
- removed joint rot1
- removed joint rot2
- added joint caja_joint: type fixed, parent base_link, child caja, origin xyz=0 0 0 rpy=0 0 0, axis 0 0 0
- added joint efector_joint: type fixed, parent prisma, child efector, origin xyz=0.00600000000004791 0 -0.0155637895736498 rpy=0 0 0, axis 0 0 0
- added joint prisma_joint: type prismatic, parent rot2, child prisma, origin xyz=0.135712735905213 0 0.23443621042635 rpy=-3.14159265358979 0 0, axis 0 0 -1, limit lower=-0.1545 upper=0 effort=1 velocity=0.15
- added joint rot1_joint: type continuous, parent base_link, child rot1, origin xyz=0 0 0.149999999999999 rpy=0 0 0.0260255178869885, axis 0 0 1, limit effort=1 velocity=0.2
- added joint rot2_joint: type continuous, parent rot1, child rot2, origin xyz=0.130000000000002 0 0.0600000000000009 rpy=0 0 -1.5707963267949, axis 0 0 1, limit effort=1 velocity=0.2

Commit message: Actualiacion de codigos trayectorias

File: Robot4/Codigo fuente/robotica/src/scara_boceto/urdf/final.urdf (robot description, URDF)
Before this commit: robot scara_boceto, 6 links, 5 joints
Links:
- link base_link: mass 0.36928 -> 0.369283968725788
- link caja: mass 0.40399 -> 0.403993820975926
- link rot1: mass 0.96022 -> 0.960224575652195
- link rot2: mass 0.8275 -> 0.827501167062165
Joints:
- joint efector_joint: limit (none) -> lower=-0.2656 effort=1 velocity=0.15; origin xyz=0.00600000000004791 0 -0.0155637895736498 rpy=0 0 0 -> xyz=0.006 0 0.29082 rpy=0 0 0
- joint prisma_joint: origin xyz=0.135712735905213 0 0.23443621042635 rpy=-3.14159265358979 0 0 -> xyz=0.13571 0 0.23444 rpy=3.1416 0 0

File: Robot4/Codigo fuente/robotica/src/scara_cajas/urdf/Ensamblaje1.urdf (robot description, URDF)
Before this commit: robot scara_cajas, 8 links, 7 joints
Joints:
- joint pris_joint: limit lower=0 upper=0.131 effort=100.0 velocity=1.0 -> lower=0 upper=0.131 effort=100.0 velocity=0.15

Commit message: Modificacion urdf

File: Robot4/Codigo fuente/robotica/src/scara_boceto/urdf/final.urdf (robot description, URDF)
Before this commit: robot scara_boceto, 6 links, 5 joints
Joints:
- joint rot1_joint: origin xyz=0 0 0.149999999999999 rpy=0 0 0.0260255178869885 -> xyz=0 0 0.149999999999999 rpy=0 0 0

Commit message: Calculos actualizados

File: Robot4/Codigo fuente/robotica/src/scara_boceto/urdf/final.urdf (robot description, URDF)
Before this commit: robot scara_boceto, 6 links, 5 joints
Joints:
- joint rot2_joint: limit effort=1 velocity=0.2 -> lower=-0.62 upper=3.3 effort=1 velocity=0.2; type continuous -> revolute
