Commit message: COnfiguracion gazebo

File: Robot4/Codigo fuente/robotica/src/scara_boceto/urdf/scara_boceto.urdf.xacro (robot description, xacro)
@@ -1,189 +1,390 @@
-<?xml version="1.0"?>
-<robot name="scara_boceto" xmlns:xacro="http://www.ros.org/wiki/xacro">
-  <xacro:arg name="controllers_yaml" default=""/>
-  <!-- DUMMY LINK Y ANCLAJE A BASE -->
-  <link name="dummy_link"/>
-  <joint name="dummy_to_base" type="fixed">
-    <parent link="dummy_link"/>
+<?xml version="1.0" encoding="utf-8"?>
+<!-- This URDF was automatically created by SolidWorks to URDF Exporter! Originally created by Stephen Brawner (brawner@gmail.com)
+     Commit Version: 1.6.0-4-g7f85cfe  Build Version: 1.6.7995.38578
+     For more information, please see http://wiki.ros.org/sw_urdf_exporter -->
+<robot xmlns:xacro="http://www.ros.org/wiki/xacro"
+       name="scara_boceto">
+  <!-- Parametros del modelo -->
+  <xacro:property name="robot_name" value="scara_boceto"/>
+  <xacro:property name="mesh_package" value="scara_boceto"/>
+  <!-- Link virtual para anclar el robot al mundo de Gazebo y evitar que se caiga -->
+  <link name="world"/>
+  <joint name="fixed_to_world" type="fixed">
+    <parent link="world"/>
     <child link="base_link"/>
     <origin xyz="0 0 0" rpy="0 0 0"/>
   </joint>
-  <!-- BASE LINK -->
-  <link name="base_link">
-    <inertial>
-      <origin xyz="0.900410418166696 0.759999999999999 0.0554005698173109" rpy="0 0 0" />
-      <mass value="0.311284852028824" />
-      <inertia
-        ixx="0.00129363756507107" ixy="1.04507041751299E-19" ixz="-4.42031795870759E-06"
-        iyy="0.00128953592508778" iyz="8.23762890581531E-18" izz="0.000695552500536542" />
-    </inertial>
-    <visual>
-      <origin xyz="0 0 0" rpy="0 0 0" />
-      <geometry><mesh filename="package://scara_boceto/meshes/base_link.STL" /></geometry>
-      <material name=""><color rgba="1 0.937254901960784 0.137254901960784 1" /></material>
-    </visual>
-    <collision>
-      <origin xyz="0 0 0" rpy="0 0 0" />
-      <geometry><mesh filename="package://scara_boceto/meshes/base_link.STL" /></geometry>
-    </collision>
-  </link>
-  <!-- EST2 LINK & JOINT -->
-  <link name="est2">
-    <inertial>
-      <origin xyz="-9.4369E-16 6.9389E-16 0.067601" rpy="0 0 0" />
-      <mass value="1.3154" />
-      <inertia
-        ixx="0.0034905" ixy="5.7965E-19" ixz="-2.8512E-17"
-        iyy="0.0034425" iyz="2.2477E-17" izz="0.0055556" />
-    </inertial>
-    <visual>
-      <origin xyz="0 0 0" rpy="0 0 0" />
-      <geometry><mesh filename="package://scara_boceto/meshes/est2.STL" /></geometry>
-      <material name=""><color rgba="1 1 1 1" /></material>
-    </visual>
-    <collision>
-      <origin xyz="0 0 0" rpy="0 0 0" />
-      <geometry><mesh filename="package://scara_boceto/meshes/est2.STL" /></geometry>
-    </collision>
-  </link>
-  <joint name="est2_joint" type="fixed">
-    <origin xyz="0.75 0.67 0" rpy="0 0 0" />
-    <parent link="base_link" />
-    <child link="est2" />
-  </joint>
-  <!-- BAN3 LINK & JOINT -->
-  <link name="ban3">
-    <inertial>
-      <origin xyz="0 2.7756E-16 0.030476" rpy="0 0 0" />
-      <mass value="0.34471" />
-      <inertia
-        ixx="0.0003887" ixy="3.5164E-21" ixz="-1.515E-20"
-        iyy="0.00038009" iyz="2.6084E-18" izz="0.00064584" />
-    </inertial>
-    <visual>
-      <origin xyz="0 0 0" rpy="0 0 0" />
-      <geometry><mesh filename="package://scara_boceto/meshes/ban3.STL" /></geometry>
-      <material name=""><color rgba="1 1 1 1" /></material>
-    </visual>
-    <collision>
-      <origin xyz="0 0 0" rpy="0 0 0" />
-      <geometry><mesh filename="package://scara_boceto/meshes/ban3.STL" /></geometry>
-    </collision>
-  </link>
-  <joint name="ban3_joint" type="fixed">
-    <origin xyz="1.08 0.88 0" rpy="0 0 0" />
-    <parent link="base_link" />
-    <child link="ban3" />
-  </joint>
-  <!-- ROT1 LINK & JOINT -->
-  <link name="rot1">
-    <inertial>
-      <origin xyz="0.065308 -2.2088E-05 0.02979" rpy="0 0 0" />
-      <mass value="0.94931" />
-      <inertia
-        ixx="0.0007704" ixy="1.575E-07" ixz="8.7916E-05"
-        iyy="0.0035092" iyz="5.2629E-07" izz="0.0036621" />
-    </inertial>
-    <visual>
-      <origin xyz="0 0 0" rpy="0 0 0" />
-      <geometry><mesh filename="package://scara_boceto/meshes/rot1.STL" /></geometry>
-      <material name=""><color rgba="1 0.93725 0.13725 1" /></material>
-    </visual>
-    <collision>
-      <origin xyz="0 0 0" rpy="0 0 0" />
-      <geometry><mesh filename="package://scara_boceto/meshes/rot1.STL" /></geometry>
-    </collision>
-  </link>
-  <joint name="rot1_joint" type="continuous">
-    <origin xyz="0.900000000000001 0.759999999999996 0.150000000000012" rpy="0 0 0" />
-    <parent link="base_link" />
-    <child link="rot1" />
-    <axis xyz="0 0 1" />
-  </joint>
-  <!-- ROT2 LINK & JOINT -->
-  <link name="rot2">
-    <inertial>
-      <origin xyz="0.039342 0.0011436 0.030461" rpy="0 0 0" />
-      <mass value="0.67755" />
-      <inertia
-        ixx="0.00055824" ixy="3.3211E-06" ixz="1.7908E-05"
-        iyy="0.0016901" iyz="1.2979E-07" izz="0.0018303" />
-    </inertial>
-    <visual>
-      <origin xyz="0 0 0" rpy="0 0 0" />
-      <geometry><mesh filename="package://scara_boceto/meshes/rot2.STL" /></geometry>
-      <material name=""><color rgba="1 0.93725 0.13725 1" /></material>
-    </visual>
-    <collision>
-      <origin xyz="0 0 0" rpy="0 0 0" />
-      <geometry><mesh filename="package://scara_boceto/meshes/rot2.STL" /></geometry>
-    </collision>
-  </link>
-  <joint name="rot2_joint" type="revolute">
-    <origin xyz="0.13 0 0.06" rpy="0 0 -1.5708" />
-    <parent link="rot1" />
-    <child link="rot2" />
-    <axis xyz="0 0 1" />
-    <limit lower="-0.5" upper="3.3" effort="100.0" velocity="1.0" />
-  </joint>
-  <!-- PRIS LINK & JOINT -->
-  <link name="pris">
-    <inertial>
-      <origin xyz="-0.01724 0.0059766 -0.2348" rpy="0 0 0" />
-      <mass value="0.10612" />
-      <inertia
-        ixx="0.00027675" ixy="9.7923E-07" ixz="2.9909E-12"
-        iyy="0.00028036" iyz="-4.1377E-12" izz="1.7505E-05" />
-    </inertial>
-    <visual>
-      <origin xyz="0 0 0" rpy="0 0 0" />
-      <geometry><mesh filename="package://scara_boceto/meshes/pris.STL" /></geometry>
-      <material name=""><color rgba="0.89804 0.91765 0.92941 1" /></material>
-    </visual>
-    <collision>
-      <origin xyz="0 0 0" rpy="0 0 0" />
-      <geometry><mesh filename="package://scara_boceto/meshes/pris.STL" /></geometry>
-    </collision>
-  </link>
-  <joint name="pris_joint" type="prismatic">
-    <origin xyz="0.13793 0.0015431 -0.048061" rpy="0 0 0" />
-    <parent link="rot2" />
-    <child link="pris" />
-    <axis xyz="0 0 -1" />
-    <limit lower="-0.131" upper="0" effort="100.0" velocity="1.0" />
-  </joint>
-  <!-- ===================== ros2_control ===================== -->
-  <ros2_control name="ScaraBocetoSystem" type="system">
-    <hardware>
-      <plugin>gz_ros2_control/GazeboSimSystem</plugin>
-    </hardware>
-    <joint name="rot1_joint">
-      <command_interface name="position">
-        <param name="min">-3.1416</param>
-        <param name="max">3.1416</param>
-      </command_interface>
-      <state_interface name="position"/>
-      <state_interface name="velocity"/>
-    </joint>
-    <joint name="rot2_joint">
-      <command_interface name="position">
-        <param name="min">-0.5</param>
-        <param name="max">3.3</param>
-      </command_interface>
-      <state_interface name="position"/>
-      <state_interface name="velocity"/>
-    </joint>
-    <joint name="pris_joint">
-      <command_interface name="position">
-        <param name="min">-0.131</param>
-        <param name="max">0</param>
-      </command_interface>
-      <state_interface name="position"/>
-      <state_interface name="velocity"/>
-    </joint>
-  </ros2_control>
-  <!-- ===================== Plugin de gz_ros2_control ===================== -->
+  <link
+    name="base_link">
+    <inertial>
+      <origin
+        xyz="7.3698831396794E-06 0.00505634398271243 0.0515191581411316"
+        rpy="0 0 0" />
+      <mass
+        value="0.369283968725788" />
+      <inertia
+        ixx="0.00143244737393282"
+        ixy="-9.70614366393655E-08"
+        ixz="-1.42672533433238E-07"
+        iyy="0.00143617210946978"
+        iyz="5.47922504699482E-06"
+        izz="0.000844588909415063" />
+    </inertial>
+    <visual>
+      <origin
+        xyz="0 0 0"
+        rpy="0 0 0" />
+      <geometry>
+        <mesh
+          filename="package://${mesh_package}/meshes/base_link.STL" />
+      </geometry>
+      <material
+        name="">
+        <color
+          rgba="0.95 0.96 0.15 1" />
+      </material>
+    </visual>
+    <collision>
+      <origin
+        xyz="0 0 0"
+        rpy="0 0 0" />
+      <geometry>
+        <mesh
+          filename="package://${mesh_package}/meshes/base_link.STL" />
+      </geometry>
+    </collision>
+  </link>
+  <link
+    name="rot1">
+    <inertial>
+      <origin
+        xyz="0.0652002981897172 2.15184196864643E-06 0.0302808417973492"
+        rpy="0 0 0" />
+      <mass
+        value="0.960224575652195" />
+      <inertia
+        ixx="0.000771578203436998"
+        ixy="-1.1237245765865E-08"
+        ixz="8.88110971334996E-05"
+        iyy="0.00351096266258402"
+        iyz="1.03264234045021E-08"
+        izz="0.00366458339979814" />
+    </inertial>
+    <visual>
+      <origin
+        xyz="0 0 0"
+        rpy="0 0 0" />
+      <geometry>
+        <mesh
+          filename="package://${mesh_package}/meshes/rot1.STL" />
+      </geometry>
+      <material
+        name="">
+        <color
+          rgba="0.95 0.96 0.15 1" />
+      </material>
+    </visual>
+    <collision>
+      <origin
+        xyz="0 0 0"
+        rpy="0 0 0" />
+      <geometry>
+        <mesh
+          filename="package://${mesh_package}/meshes/rot1.STL" />
+      </geometry>
+    </collision>
+  </link>
+  <joint
+    name="rot1_joint"
+    type="continuous">
+    <origin
+      xyz="0 0 0.149999999999999"
+      rpy="0 0 0" />
+    <parent
+      link="base_link" />
+    <child
+      link="rot1" />
+    <axis
+      xyz="0 0 1" />
+    <limit
+      effort="10"
+      velocity="2.0" />
+    <dynamics
+      damping="0.5"
+      friction="0.1" />
+  </joint>
+  <link
+    name="rot2">
+    <inertial>
+      <origin
+        xyz="0.0545562991886573 0.00420940477256759 0.0442384523201031"
+        rpy="0 0 0" />
+      <mass
+        value="0.827501167062165" />
+      <inertia
+        ixx="0.000723895006460007"
+        ixy="-2.0619565009593E-06"
+        ixz="2.00409100148053E-05"
+        iyy="0.00244181599386376"
+        iyz="-6.47140205432564E-08"
+        izz="0.00249469873379645" />
+    </inertial>
+    <visual>
+      <origin
+        xyz="0 0 0"
+        rpy="0 0 0" />
+      <geometry>
+        <mesh
+          filename="package://${mesh_package}/meshes/rot2.STL" />
+      </geometry>
+      <material
+        name="">
+        <color
+          rgba="0.50 0.50 0.51 1" />
+      </material>
+    </visual>
+    <collision>
+      <origin
+        xyz="0 0 0"
+        rpy="0 0 0" />
+      <geometry>
+        <mesh
+          filename="package://${mesh_package}/meshes/rot2.STL" />
+      </geometry>
+    </collision>
+  </link>
+  <joint
+    name="rot2_joint"
+    type="revolute">
+    <origin
+      xyz="0.130000000000002 0 0.0600000000000009"
+      rpy="0 0 -1.5707963267949" />
+    <parent
+      link="rot1" />
+    <child
+      link="rot2" />
+    <axis
+      xyz="0 0 1" />
+    <limit
+      lower="-0.62"
+      upper="3.3"
+      effort="10"
+      velocity="2.0" />
+    <dynamics
+      damping="0.5"
+      friction="0.1" />
+  </joint>
+  <link
+    name="prisma">
+    <inertial>
+      <origin
+        xyz="-0.00968954429107238 -8.70297020284794E-05 0.00763925129938392"
+        rpy="0 0 0" />
+      <mass
+        value="0.0482530059600755" />
+      <inertia
+        ixx="3.78986465008096E-05"
+        ixy="1.55038979176541E-10"
+        ixz="-4.10087887988017E-11"
+        iyy="3.08945956859896E-05"
+        iyz="3.63265544654102E-20"
+        izz="9.67997761427531E-06" />
+    </inertial>
+    <visual>
+      <origin
+        xyz="0 0 0"
+        rpy="0 0 0" />
+      <geometry>
+        <mesh
+          filename="package://${mesh_package}/meshes/prisma.STL" />
+      </geometry>
+      <material
+        name="">
+        <color
+          rgba="0.792156862745098 0.819607843137255 0.933333333333333 1" />
+      </material>
+    </visual>
+    <collision>
+      <origin
+        xyz="0 0 0"
+        rpy="0 0 0" />
+      <geometry>
+        <mesh
+          filename="package://${mesh_package}/meshes/prisma.STL" />
+      </geometry>
+    </collision>
+  </link>
+  <joint
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